File: practice/practice.kicad_sch (KiCad schematic)
At the start: 4 parts

Commit message: 修改 R1 阻值
Parts:
- R1: value 220 -> 1000
Changed lines of the file:
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@@
     (in_bom yes) (on_board yes) (fields_autoplaced)
     (property "Reference" "R1" (id 0) (at 134.62 82.55 90))
-    (property "Value" "220" (id 1) (at 134.62 85.09 90))
+    (property "Value" "1000" (id 1) (at 134.62 85.09 90))
     (property "Footprint" "Resistor_THT:R_Axial_DIN0207_L6.3mm_D2.5mm_P10.16mm_Horizontal" (id 2) (at 134.62 90.678 90)
       (effects (font (size 1.27 1.27)) hide)
@@
     )
     (path "/2de85b8a-5fc0-4e21-ad52-2cca4d4125c0"
-      (reference "R1") (unit 1) (value "220") (footprint "Resistor_THT:R_Axial_DIN0207_L6.3mm_D2.5mm_P10.16mm_Horizontal")
+      (reference "R1") (unit 1) (value "1000") (footprint "Resistor_THT:R_Axial_DIN0207_L6.3mm_D2.5mm_P10.16mm_Horizontal")
     )
     (path "/7d830e22-5b15-4106-abc9-fcdc42c188aa"
